Commit message: joystick control working, visual of camera, but still seeing mount hen driving

File: turtlebot3_description/urdf/turtlebot3_waffle_pi.urdf.xacro (robot description, xacro)
@@ -229,8 +229,8 @@
   <gazebo reference="scan_link">
     <xacro:ray_sensor sensor_name="scan" gazebo="ignition"
-                  update_rate="10.0" visualize="true"
-                  h_samples="360" h_res="1.0" h_min_angle="0.000" h_max_angle="6.280000"
-                  r_min="0.164" r_max="20.0" r_res="0.01">
-                  <plugin name="dummy" filename="dummyfile"></plugin>
+      update_rate="10.0" visualize="true"
+      h_samples="360" h_res="1.0" h_min_angle="0.000" h_max_angle="6.280000"
+      r_min="0.164" r_max="20.0" r_res="0.01">
+      <plugin name="dummy" filename="dummyfile"></plugin>
     </xacro:ray_sensor>
     <xacro:material_darkgray />
@@ -240,5 +240,5 @@
   </gazebo>
   <joint name="camera_joint" type="fixed">
-    <origin xyz="0.073 -0.011 0.084" rpy="0 0 0" />
+    <origin xyz="0.083 -0.0 0.097" rpy="0 0 0" />
     <parent link="base_link" />
     <child link="camera_link" />
@@ -246,16 +246,28 @@
   <link name="camera_link">
     <collision>
-      <origin xyz="0.005 0.011 0.013" rpy="0 0 0" />
+      <origin xyz="0.005 0.0 0.013" rpy="0 0 0" />
       <geometry>
         <box size="0.015 0.030 0.027" />
       </geometry>
     </collision>
+    <visual>
+      <geometry>
+        <box size="0.015 0.03 0.027" />
+      </geometry>
+    </visual>
   </link>
   <joint name="camera_rgb_joint" type="fixed">
-    <origin xyz="0.003 0.011 0.009" rpy="0 0 0" />
+    <origin xyz="0.01 0.0 0.0" rpy="0 0 0" />
     <parent link="camera_link" />
     <child link="camera_rgb_frame" />
   </joint>
-  <link name="camera_rgb_frame" />
+  <link name="camera_rgb_frame">
+    <!-- <visual>
+    <origin xyz="0.0 0.0 0.0" rpy="0 1.57 0" />
+      <geometry>
+        <cylinder radius="0.007" length="0.005" />
+      </geometry>
+    </visual> -->
+  </link>
   <joint name="camera_rgb_optical_joint" type="fixed">
     <origin xyz="0 0 0" rpy="-1.57 0 -1.57" />
@@ -364,5 +376,5 @@
       <topic>rgbd_camera</topic>
     </sensor>
-    <xacro:material_darkgray/>
+    <xacro:material_darkgray />
   </gazebo>
 </robot>
